File: eagle/RN42/RN42_breakout.brd (EAGLE design)
At the start: 38.8 x 22.9 mm, 24 parts, among them T1 N-MOSFET, T2 N-MOSFET, T3 LM3480IM4

Commit message: RN42: update some values.
Parts:
- C1: value (none) -> 1uF
- C2, C3: value (none) -> 0.1uF

Commit message: Update RN42 breakout board.
Moved the capacitor for the LDO near to the LDO and the decoupling
capacitor near the VCC of the main chip (originally C1 and C3 where
exchanged).
Parts:
- moved C3 9.99 mm to (28.2, 3.05), turned to 270 degrees
- moved C1 8.74 mm to (16.3, 1.78), turned to 180 degrees
- moved L3 2.54 mm to (24.1, 2.79)
- moved R7 2.54 mm to (24.1, 5.84)
Routing:
- net 3V3: track 77.5 -> 81.9 mm
Changed lines of the file:
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@@
 <text x="32.258" y="7.874" size="1.016" layer="21" font="vector" ratio="16">GND</text>
 <text x="32.004" y="18.288" size="1.016" layer="21" font="vector" ratio="16">3V3</text>
-<text x="23.114" y="2.286" size="1.016" layer="25" font="vector" ratio="16">PWR</text>
+<text x="20.574" y="2.286" size="1.016" layer="25" font="vector" ratio="16">PWR</text>
 <text x="32.258" y="10.414" size="1.016" layer="21" font="vector" ratio="16">VCC</text>
-<wire x1="22.606" y1="3.81" x2="22.352" y2="3.81" width="0.4064" layer="21"/>
-<wire x1="22.352" y1="3.81" x2="22.352" y2="1.524" width="0.4064" layer="21"/>
-<wire x1="22.352" y1="1.524" x2="22.606" y2="1.524" width="0.4064" layer="21"/>
-<wire x1="27.686" y1="1.524" x2="27.94" y2="1.524" width="0.4064" layer="21"/>
-<wire x1="27.94" y1="1.524" x2="27.94" y2="3.81" width="0.4064" layer="21"/>
-<wire x1="27.94" y1="3.81" x2="27.686" y2="3.81" width="0.4064" layer="21"/>
+<wire x1="20.066" y1="3.81" x2="19.812" y2="3.81" width="0.4064" layer="21"/>
+<wire x1="19.812" y1="3.81" x2="19.812" y2="1.524" width="0.4064" layer="21"/>
+<wire x1="19.812" y1="1.524" x2="20.066" y2="1.524" width="0.4064" layer="21"/>
+<wire x1="25.146" y1="1.524" x2="25.4" y2="1.524" width="0.4064" layer="21"/>
+<wire x1="25.4" y1="1.524" x2="25.4" y2="3.81" width="0.4064" layer="21"/>
+<wire x1="25.4" y1="3.81" x2="25.146" y2="3.81" width="0.4064" layer="21"/>
 <hole x="2.54" y="21.59" drill="1.2"/>
 <hole x="2.54" y="1.27" drill="1.2"/>
@@
 <attribute name="VALUE" x="21.463" y="16.129" size="1.27" layer="27" rot="R270"/>
 </element>
-<element name="C1" library="rcl" package="C0603" value="1uF" x="23.368" y="6.858" smashed="yes" rot="R270">
-<attribute name="NAME" x="24.003" y="6.985" size="1.016" layer="25" font="vector" ratio="16" rot="R270"/>
-<attribute name="VALUE" x="21.463" y="7.493" size="1.27" layer="27" rot="R270"/>
+<element name="C1" library="rcl" package="C0603" value="1uF" x="16.256" y="1.778" smashed="yes" rot="R180">
+<attribute name="NAME" x="16.383" y="1.143" size="1.016" layer="25" font="vector" ratio="16" rot="R180"/>
+<attribute name="VALUE" x="16.891" y="3.683" size="1.27" layer="27" rot="R180"/>
 </element>
 <element name="J1" library="SparkFun-Connectors" package="1X07" value="" x="36.576" y="3.302" smashed="yes" rot="R90">
@@
 </element>
 <element name="C2" library="SparkFun-Passives" package="0603-CAP" value="0.1uF" x="30.988" y="3.048" smashed="yes" rot="R270">
-<attribute name="NAME" x="28.956" y="3.937" size="1.016" layer="21" font="vector" ratio="16" rot="R270"/>
+<attribute name="NAME" x="30.099" y="4.826" size="1.016" layer="21" font="vector" ratio="16"/>
 <attribute name="VALUE" x="29.845" y="4.064" size="0.4064" layer="27" font="vector" rot="R270"/>
 </element>
-<element name="C3" library="SparkFun-Passives" package="0603-CAP" value="0.1uF" x="18.288" y="1.778" smashed="yes">
-<attribute name="NAME" x="17.399" y="2.54" size="1.016" layer="25" font="vector" ratio="16"/>
-<attribute name="VALUE" x="17.272" y="0.635" size="0.4064" layer="27" font="vector"/>
+<element name="C3" library="SparkFun-Passives" package="0603-CAP" value="0.1uF" x="28.194" y="3.048" smashed="yes" rot="R270">
+<attribute name="NAME" x="27.305" y="4.826" size="1.016" layer="25" font="vector" ratio="16"/>
+<attribute name="VALUE" x="27.051" y="4.064" size="0.4064" layer="27" font="vector" rot="R270"/>
 </element>
 <element name="T2" library="GeekAmmo" package="SOT23-3" value="N-MOSFET" x="27.178" y="19.304" smashed="yes" rot="R270">
@@
 <attribute name="VALUE" x="7.62" y="22.479" size="1.27" layer="27" rot="R180"/>
 </element>
-<element name="R7" library="rcl" package="R0603" value="1k" x="26.67" y="5.842" smashed="yes" rot="R90">
-<attribute name="NAME" x="28.829" y="4.953" size="1.016" layer="25" font="vector" ratio="16" rot="R90"/>
-<attribute name="VALUE" x="28.575" y="5.207" size="1.27" layer="27" rot="R90"/>
-</element>
-<element name="L3" library="led" package="CHIPLED_0603" value="" x="26.67" y="2.794" smashed="yes" rot="R180">
-<attribute name="VALUE" x="24.765" y="4.064" size="1.27" layer="27" rot="R270"/>
+<element name="R7" library="rcl" package="R0603" value="1k" x="24.13" y="5.842" smashed="yes" rot="R90">
+<attribute name="NAME" x="26.289" y="4.953" size="1.016" layer="25" font="vector" ratio="16" rot="R90"/>
+<attribute name="VALUE" x="26.035" y="5.207" size="1.27" layer="27" rot="R90"/>
+</element>
+<element name="L3" library="led" package="CHIPLED_0603" value="" x="24.13" y="2.794" smashed="yes" rot="R180">
+<attribute name="VALUE" x="22.225" y="4.064" size="1.27" layer="27" rot="R270"/>
 </element>
 <element name="MASTER" library="jumper" package="SJ" value="" x="3.81" y="7.874" smashed="yes" rot="MR90">
@@
 <contactref element="U$1" pad="11"/>
 <contactref element="STATUS" pad="A"/>
-<wire x1="23.368" y1="8.89" x2="23.368" y2="7.708" width="0.4064" layer="1"/>
 <wire x1="17.78" y1="8.89" x2="23.368" y2="8.89" width="0.4064" layer="16"/>
 <wire x1="16.764" y1="8.382" x2="17.78" y2="8.89" width="0.4064" layer="16"/>
@@
 <contactref element="T1" pad="1"/>
 <contactref element="R4" pad="2"/>
-<wire x1="17.438" y1="1.778" x2="17.084" y2="2.894" width="0.4064" layer="1"/>
-<wire x1="17.084" y1="2.894" x2="17.084" y2="4.576" width="0.4064" layer="1"/>
 <wire x1="29.022" y1="7.382" x2="27.768" y2="8.636" width="0.4064" layer="1"/>
 <wire x1="27.768" y1="8.636" x2="26.67" y2="8.636" width="0.4064" layer="1"/>
@@
 <wire x1="23.026" y1="20.066" x2="23.622" y2="20.154" width="0.4064" layer="1"/>
 <contactref element="R7" pad="2"/>
-<wire x1="26.67" y1="6.692" x2="26.67" y2="8.636" width="0.4064" layer="1"/>
+<wire x1="24.13" y1="6.692" x2="26.67" y2="8.636" width="0.4064" layer="1"/>
 <contactref element="MASTER" pad="2"/>
 <wire x1="9.398" y1="10.414" x2="14.732" y2="10.414" width="0.4064" layer="16"/>
@@
 <wire x1="28.448" y1="20.574" x2="26.498" y2="20.574" width="0.4064" layer="1"/>
 <wire x1="26.498" y1="20.574" x2="26.178" y2="20.254" width="0.4064" layer="1"/>
+<wire x1="28.194" y1="3.898" x2="29.022" y2="3.898" width="0.4064" layer="1"/>
+<wire x1="29.022" y1="3.898" x2="29.022" y2="7.382" width="0.4064" layer="1"/>
+<wire x1="17.106" y1="1.778" x2="17.084" y2="1.778" width="0.4064" layer="1"/>
+<wire x1="17.084" y1="1.778" x2="17.084" y2="4.576" width="0.4064" layer="1"/>
 </signal>
 <signal name="TXH">
@@
 <contactref element="R7" pad="1"/>
 <contactref element="L3" pad="A"/>
-<wire x1="26.67" y1="4.992" x2="26.67" y2="3.544" width="0.4064" layer="1"/>
+<wire x1="24.13" y1="4.992" x2="24.13" y2="3.544" width="0.4064" layer="1"/>
 </signal>
 <signal name="AUTODISCOVERY">
